Commit message: Updated URDF to properly use xacro

File: src/roomba_891_py/description/drivebase.xacro (robot description, xacro)
@@ -1,13 +1,13 @@
 <?xml version="1.0"?>
 <robot xmlns:xacro="http://www.ros.org/wiki/xacro">
+    <xacro:include filename="dimensions.xacro"/>
+    <xacro:include filename="materials.xacro"/>
     <link name="chassis_link">
         <visual>
             <origin xyz="0.0 0.0 0.0375"/>
             <geometry>
-                <cylinder radius="0.170" length="0.075"/>
+                <cylinder radius="${chassis_radius}" length="${chassis_height}"/>
             </geometry>
-            <material name="gray">
-                <color rgba="0.5 0.5 0.5 1"/>
-            </material>
+            <material name="grey"/>
         </visual>
     </link>
@@ -16,8 +16,6 @@
             <origin xyz="0.0 0.0 0.0"/>
             <geometry>
-                <cylinder radius="0.0375" length="0.016"/>
-                <material>
-                    <color rgba="1 0.0 0.0 1"/>
-                </material>
+                <cylinder radius="${wheel_radius}" length="${wheel_thickness}"/>
+                <material name="red"/>
             </geometry>
         </visual>
@@ -27,8 +25,6 @@
             <origin xyz="0.0 0.0 0.0"/>
             <geometry>
-                <cylinder radius="0.0375" length="0.016"/>
-                <material>
-                    <color rgba="1 0.0 0.0 1"/>
-                </material>
+                <cylinder radius="${wheel_radius}" length="${wheel_thickness}"/>
+                <material name="red"/>
             </geometry>
         </visual>
@@ -38,9 +34,7 @@
             <origin xyz="0.0 0.0 0.0"/>
             <geometry>
-                <sphere radius="0.047"/>
+                <sphere radius="${caster_radius}"/>
             </geometry>
-            <material name="white">
-                <color rgba="1.0 1.0 1.0 1.0"/>
-            </material>
+            <material name="red"/>
         </visual>
     </link>
@@ -52,5 +46,5 @@
     </joint>
     <joint name="left_wheel_joint" type="continuous">
-        <origin xyz="0.0 0.110 0.0" rpy="${pi/2} 0.0 0.0"/>
+        <origin xyz="0.0 ${wheel_offset} 0.0" rpy="${pi/2} 0.0 0.0"/>
         <parent link="chassis_link"/>
         <child link="left_wheel"/>
@@ -58,5 +52,5 @@
     </joint>
     <joint name="right_wheel_joint" type="continuous">
-        <origin xyz="0.0 -0.110 0.0" rpy="${pi/2} 0.0 0.0"/>
+        <origin xyz="0.0 -${wheel_offset} 0.0" rpy="${pi/2} 0.0 0.0"/>
         <parent link="chassis_link"/>
         <child link="right_wheel"/>

Commit message: chore: Add macros.xacro for solid sphere and solid cylinder inertia calculations

File: src/roomba_891_py/description/drivebase.xacro (robot description, xacro)
@@ -3,4 +3,5 @@
     <xacro:include filename="dimensions.xacro"/>
     <xacro:include filename="materials.xacro"/>
+    <xacro:include filename="macros.xacro"/>
     <link name="chassis_link">
         <visual>
@@ -11,4 +12,14 @@
             <material name="grey"/>
         </visual>
+        <collision>
+            <origin xyz="0.0 0.0 0.0375"/>
+            <geometry>
+                <cylinder radius="${chassis_radius}" length="${chassis_height}"/>
+            </geometry>
+        </collision>
+        <inertial>
+            <mass value="2.95"/>
+            <xacro:solid_cylinder_inertia m="2.95" r="${chassis_radius}" h="${chassis_height}"/>
+        </inertial>
     </link>
     <link name="left_wheel">
@@ -17,7 +28,16 @@
             <geometry>
                 <cylinder radius="${wheel_radius}" length="${wheel_thickness}"/>
-                <material name="red"/>
             </geometry>
+            <material name="red"/>
         </visual>
+        <collision>
+            <geometry>
+                <cylinder radius="${wheel_radius}" length="${wheel_thickness}"/>
+            </geometry>
+        </collision>
+        <inertial>
+            <mass value="0.226796"/>
+            <xacro:solid_cylinder_inertia m="0.226796" r="${wheel_radius}" h="${wheel_thickness}"/>
+        </inertial>
     </link>
     <link name="right_wheel">
@@ -26,7 +46,16 @@
             <geometry>
                 <cylinder radius="${wheel_radius}" length="${wheel_thickness}"/>
-                <material name="red"/>
             </geometry>
+            <material name="red"/>
         </visual>
+        <collision>
+            <geometry>
+                <cylinder radius="${wheel_radius}" length="${wheel_thickness}"/>
+            </geometry>
+        </collision>
+        <inertial>
+            <mass value="0.226796"/>
+            <xacro:solid_cylinder_inertia m="0.226796" r="${wheel_radius}" h="${wheel_thickness}"/>
+        </inertial>
     </link>
     <link name="caster_wheel">
@@ -38,4 +67,13 @@
             <material name="red"/>
         </visual>
+        <collision>
+            <geometry>
+                <sphere radius="${caster_radius}"/>
+            </geometry>
+        </collision>
+        <inertial>
+            <mass value="0.05"/>
+            <xacro:solid_sphere_inertia m="0.05" r="${caster_radius}"/>
+        </inertial>
     </link>
     <joint name="caster_joint" type="continuous">
