Commit message: added diffdrive plugin to fix gravity (didnt work)

File: src/roomba_891_py/description/dimensions.xacro (robot description, xacro)
@@ -5,5 +5,5 @@
     <xacro:property name="wheel_radius" value="0.0375"/>
     <xacro:property name="wheel_thickness" value="0.016"/>
-    <xacro:property name="caster_radius" value="0.047"/>
+    <xacro:property name="caster_radius" value="0.0375"/>
     <xacro:property name="wheel_offset" value="0.110"/>
 </robot>

File: src/roomba_891_py/description/gazebo.xacro (robot description, xacro)
@@ -20,4 +20,21 @@
             <joint>right_wheel_joint</joint>
         </plugin>
+        <plugin filename="gz-sim-diff-drive-system" name="gz::sim::systems::DiffDrive">
+            <!-- Remove <ros> tag. -->
+            <!-- wheels -->
+            <left_joint>left_wheel_joint</left_joint>
+            <right_joint>right_wheel_joint</right_joint>
+            <!-- kinematics -->
+            <wheel_separation>0.220</wheel_separation>
+            <wheel_radius>0.0375</wheel_radius> <!-- computed from <wheel_diameter> in the original plugin-->
+            <!-- limits -->
+            <max_linear_acceleration>0.033</max_linear_acceleration> <!-- computed from <max_linear_acceleration> in the original plugin-->
+            <topic>cmd_vel</topic> <!-- from <commant_topic> -->
+            <odom_topic>odom</odom_topic> <!-- from <odometry_topic> -->
+            <frame_id>world</frame_id> <!-- from <odometry_frame> -->
+            <child_frame_id>base_footprint</child_frame_id> <!-- from <robot_base_frame> -->
+            <odom_publisher_frequency>30</odom_publisher_frequency> <!-- from <update_rate>-->
+            <tf_topic>/tf</tf_topic> <!-- Short topic name for tf output -->
+          </plugin>
     </gazebo>
 </robot>

File: src/roomba_891_py/description/robot_base.urdf.xacro (robot description, xacro)
@@ -4,5 +4,5 @@
     <xacro:include filename="drivebase.xacro"/>
     <joint name="base_joint" type="fixed">
-        <origin xyz="0.0 0.0 0.016" rpy="0.0 0.0 0.0"/>
+        <origin xyz="0.0 0.0 ${wheel_radius}" rpy="0.0 0.0 0.0"/>
         <parent link="world"/>
         <child link="chassis_link"/>
